File: awuita.sch (KiCad schematic (older format))
At the start: 146 parts, among them SW1 SW_Push, SW2 Rotary_Encoder, U1 ATmega32U4-AU, Y1 Crystal_GND24_Small

Commit message: Updates on schematic
Parts:
- removed C1, C2: 22pF, symbol Device:C_Small
- removed R1, R2: 22, symbol Device:R_Small
- removed R3: 10k, symbol Device:R_Small
- removed SW1: SW_Push, symbol Switch:SW_Push
- removed Y1: Crystal_GND24_Small, symbol Device:Crystal_GND24_Small
- added C? (x2): 22p, symbol Device:C_Small
- added C?: 1u, symbol Device:C_Small
- added F?: 500m, symbol Device:Polyfuse_Small
- added J?: AVR-ISP-6, symbol Connector:AVR-ISP-6
- added R?: 10k, symbol Device:R_Small
- added R? (x2): 22, symbol Device:R_Small
- added R? (x2): 5.1K, symbol Device:R_Small
- added SW?: Reset_SW, symbol Switch:SW_Push
- added U?: PRTR5V0U2X, symbol random-keyboard-parts:PRTR5V0U2X
- added USB?: HRO-TYPE-C-31-M-12, symbol Type-C:HRO-TYPE-C-31-M-12
- added Y?: Crystal_GND24_Small, symbol Device:Crystal_GND24_Small
Connections:
- net labels added: D+, D-, MISO, MOSI, RESET, SCK, VCC, XTAL1, XTAL2
- wire segments 259 -> 301
- no-connect marks 0 -> 2
Other:
- moved on the sheet: C3, C4, C5, C6, R4, U1
